Commit message: Update vx300s.xacro

File: urdf/vx300s.xacro (robot description, xacro)
@@ -24,3 +24,69 @@
 		</plugin>
 	</gazebo>
+<link name="top_CAM_1">
+  <visual>
+    <geometry>
+      <box size="0.05 0.05 0.05"/>
+    </geometry>
+    <material name="interbotix_black" />
+  </visual>
+  <collision>
+    <geometry>
+      <box size="0.05 0.05 0.05"/>
+    </geometry>
+  </collision>
+  <inertial>
+    <mass value="0.1"/>
+    <inertia ixx="0.0001" ixy="0.0" ixz="0.0"
+             iyy="0.0001" iyz="0.0"
+             izz="0.0001"/>
+  </inertial>
+</link>
+<!-- Joint connecting camera to base_link -->
+<joint name="top_CAM_joint" type="fixed">
+  <parent link="world"/>
+  <child link="top_CAM_1"/>
+  <origin xyz="0.0 0.0 0.8" rpy="0.0 0.0 0"/>
+</joint>
+    <gazebo reference="top_CAM_1">
+  <sensor name="top_zed_CAM" type="camera">
+    <always_on>true</always_on>
+    <update_rate>5</update_rate>
+    <!--pose>0.05 0 0 0 0 0.15</pose-->
+    <visualize>true</visualize>
+    <topic>/top_cam/image_raw</topic>
+    <gz_frame_id>top_CAM_1</gz_frame_id>
+    <camera name="top_zed_CAM">
+      <horizontal_fov>1.047</horizontal_fov>
+      <camera_info_topic>/top_cam/camera_info</camera_info_topic>
+      <distortion>
+        <k1>0.01</k1>
+        <k2>0.01</k2>
+        <k3>0.01</k3>
+        <p1>0.001</p1>
+        <p2>0.001</p2>
+      </distortion>
+      <image>
+        <width>244</width>
+        <height>244</height>
+        <format>R8G8B8</format>
+      </image>
+      <clip>
+        <near>0.01</near>
+        <far>5.0</far>
+      </clip>
+      <noise>
+        <type>gaussian</type>
+        <mean>0.01</mean>
+        <stddev>0.005</stddev>
+      </noise>
+       <!--depth_camera>
+        <clip>
+          <near>0.01</near>
+          <far>5</far>
+        </clip>
+      </depth_camera-->
+    </camera>
+  </sensor>
+</gazebo>
 </robot>

Commit message: latest working version

File: urdf/vx300s.xacro (robot description, xacro)
@@ -24,5 +24,5 @@
 		</plugin>
 	</gazebo>
-<link name="top_CAM_1">
+<link name="high_CAM_1">
   <visual>
     <geometry>
@@ -44,20 +44,20 @@
 </link>
 <!-- Joint connecting camera to base_link -->
-<joint name="top_CAM_joint" type="fixed">
+<joint name="high_CAM_joint" type="fixed">
   <parent link="world"/>
-  <child link="top_CAM_1"/>
+  <child link="high_CAM_1"/>
   <origin xyz="0.0 0.0 0.8" rpy="0.0 0.0 0"/>
 </joint>
-    <gazebo reference="top_CAM_1">
-  <sensor name="top_zed_CAM" type="camera">
+    <gazebo reference="high_CAM_1">
+  <sensor name="high_zed_CAM" type="camera">
     <always_on>true</always_on>
-    <update_rate>5</update_rate>
+    <update_rate>25</update_rate>
     <!--pose>0.05 0 0 0 0 0.15</pose-->
     <visualize>true</visualize>
-    <topic>/top_cam/image_raw</topic>
-    <gz_frame_id>top_CAM_1</gz_frame_id>
-    <camera name="top_zed_CAM">
+    <topic>/high_cam/image_raw</topic>
+    <gz_frame_id>high_CAM_1</gz_frame_id>
+    <camera name="high_zed_CAM">
       <horizontal_fov>1.047</horizontal_fov>
-      <camera_info_topic>/top_cam/camera_info</camera_info_topic>
+      <camera_info_topic>/high_cam/camera_info</camera_info_topic>
       <distortion>
         <k1>0.01</k1>
@@ -68,6 +68,72 @@
       </distortion>
       <image>
-        <width>244</width>
-        <height>244</height>
+        <width>224</width>
+        <height>224</height>
+        <format>R8G8B8</format>
+      </image>
+      <clip>
+        <near>0.01</near>
+        <far>5.0</far>
+      </clip>
+      <noise>
+        <type>gaussian</type>
+        <mean>0.01</mean>
+        <stddev>0.005</stddev>
+      </noise>
+       <!--depth_camera>
+        <clip>
+          <near>0.01</near>
+          <far>5</far>
+        </clip>
+      </depth_camera-->
+    </camera>
+  </sensor>
+</gazebo>
+<link name="low_CAM_1">
+  <visual>
+    <geometry>
+      <box size="0.05 0.05 0.05"/>
+    </geometry>
+    <material name="interbotix_black" />
+  </visual>
+  <collision>
+    <geometry>
+      <box size="0.05 0.05 0.05"/>
+    </geometry>
+  </collision>
+  <inertial>
+    <mass value="0.1"/>
+    <inertia ixx="0.0001" ixy="0.0" ixz="0.0"
+             iyy="0.0001" iyz="0.0"
+             izz="0.0001"/>
+  </inertial>
+</link>
+<!-- Joint connecting camera to base_link -->
+<joint name="low_CAM_joint" type="fixed">
+  <parent link="world"/>
+  <child link="low_CAM_1"/>
+  <origin xyz="0.0 0.0 0.8" rpy="0.0 0.0 0"/>
+</joint>
+    <gazebo reference="low_CAM_1">
+  <sensor name="low_zed_CAM" type="camera">
+    <always_on>true</always_on>
+    <update_rate>25</update_rate>
+    <!--pose>0.05 0 0 0 0 0.15</pose-->
+    <visualize>true</visualize>
+    <topic>/low_cam/image_raw</topic>
+    <gz_frame_id>low_CAM_1</gz_frame_id>
+    <camera name="low_zed_CAM">
+      <horizontal_fov>1.047</horizontal_fov>
+      <camera_info_topic>/low_cam/camera_info</camera_info_topic>
+      <distortion>
+        <k1>0.01</k1>
+        <k2>0.01</k2>
+        <k3>0.01</k3>
+        <p1>0.001</p1>
+        <p2>0.001</p2>
+      </distortion>
+      <image>
+        <width>224</width>
+        <height>224</height>
         <format>R8G8B8</format>
       </image>

File: urdf/vx300s_macro.xacro (robot description, xacro)
@@ -402,9 +402,9 @@
     <!--pose>0.05 0 0 0 0 0.15</pose-->
     <visualize>true</visualize>
-    <topic>/${prefix}_cam/image_raw</topic>
+    <topic>/${prefix}_cam_arm/image_raw</topic>
     <gz_frame_id>${prefix}_CAM_1</gz_frame_id>
     <camera name="${prefix}_zed_CAM">
       <horizontal_fov>1.047</horizontal_fov>
-      <camera_info_topic>/${prefix}_cam/camera_info</camera_info_topic>
+      <camera_info_topic>/${prefix}_cam_arm/camera_info</camera_info_topic>
       <distortion>
         <k1>0.01</k1>
@@ -415,6 +415,6 @@
       </distortion>
       <image>
-        <width>244</width>
-        <height>244</height>
+        <width>224</width>
+        <height>224</height>
         <format>R8G8B8</format>
       </image>

Commit message: update 1

File: urdf/vx300s.xacro (robot description, xacro)
@@ -9,13 +9,42 @@
   <xacro:vx300s prefix="$(arg right_prefix)" hw_interface="hardware_interface/EffortJointInterface" />
   <link name="world" />
+  <link name="table">
+    <visual>
+      <origin xyz="0 0 0.0125" rpy="0 0 0"/>
+      <geometry>
+        <box size="1.22 0.7 0.025"/>
+      </geometry>
+      <material name="white">
+        <color rgba="1.0 1.0 1.0 1.0"/>
+      </material>
+    </visual>
+    <collision>
+      <origin xyz="0 0 0.0125" rpy="0 0 0"/>
+      <geometry>
+        <box size="1.22 0.7 0.05"/>
+      </geometry>
+    </collision>
+    <inertial>
+      <origin xyz="0 0 0.0125" rpy="0 0 0"/>
+      <mass value="5.0"/>
+      <inertia ixx="0.1" ixy="0.0" ixz="0.0"
+               iyy="0.1" iyz="0.0"
+               izz="0.1"/>
+    </inertial>
+  </link>
+  <joint name="table_to_world" type="fixed">
+    <parent link="world" />
+     <child link="table" />
+    <origin xyz="0 0 0" rpy=" 0 0 0"/>
+  </joint>
   <joint name="$(arg left_prefix)_to_world" type="fixed">
-    <parent link="world" />
+    <parent link="table" />
     <child link="$(arg left_prefix)_base_link" />
-    <origin xyz="-0.4 0 0.7" rpy=" 0 0 1.57"/>
+    <origin xyz="-0.6 0 0.025" rpy=" 0 0 0"/>
   </joint>
   <joint name="$(arg right_prefix)_to_world" type="fixed">
-    <parent link="world" />
+    <parent link="table" />
     <child link="$(arg right_prefix)_base_link" />
-    <origin xyz="0.4 0 0.7" rpy=" 0 0 1.57"/>
+    <origin xyz="0.6 0 0.025" rpy=" 0 0 -3.14"/>
   </joint>
   <gazebo>
@@ -23,4 +52,11 @@
    			<render_engine>ogre2</render_engine>
 		</plugin>
+		<plugin filename="gz-sim-pose-publisher-system" name="gz::sim::systems::PosePublisher">
+           <publish_link_pose>true</publish_link_pose>
+           <publish_nested_model_pose>true</publish_nested_model_pose>
+           <use_pose_vector_msg>false</use_pose_vector_msg>
+           <static_publisher>true</static_publisher>
+           <static_update_frequency>1</static_update_frequency>
+        </plugin>
 	</gazebo>
 <link name="high_CAM_1">
@@ -47,11 +83,11 @@
   <parent link="world"/>
   <child link="high_CAM_1"/>
-  <origin xyz="0.0 0.0 0.8" rpy="0.0 0.0 0"/>
+  <origin xyz="0.0 -0.2 1.2" rpy="0.0 1.57 0.0"/>
 </joint>
     <gazebo reference="high_CAM_1">
   <sensor name="high_zed_CAM" type="camera">
     <always_on>true</always_on>
-    <update_rate>25</update_rate>
-    <!--pose>0.05 0 0 0 0 0.15</pose-->
+    <update_rate>50</update_rate>
+    <pose>0 0 0 0 0 0</pose>
     <visualize>true</visualize>
     <topic>/high_cam/image_raw</topic>
@@ -68,6 +104,6 @@
       </distortion>
       <image>
-        <width>224</width>
-        <height>224</height>
+        <width>640</width>
+        <height>480</height>
         <format>R8G8B8</format>
       </image>
@@ -90,4 +126,5 @@
   </sensor>
 </gazebo>
+<!--
 <link name="low_CAM_1">
   <visual>
@@ -109,5 +146,4 @@
   </inertial>
 </link>
-<!-- Joint connecting camera to base_link -->
 <joint name="low_CAM_joint" type="fixed">
   <parent link="world"/>
@@ -119,5 +155,4 @@
     <always_on>true</always_on>
     <update_rate>25</update_rate>
-    <!--pose>0.05 0 0 0 0 0.15</pose-->
     <visualize>true</visualize>
     <topic>/low_cam/image_raw</topic>
@@ -147,12 +182,7 @@
         <stddev>0.005</stddev>
       </noise>
-       <!--depth_camera>
-        <clip>
-          <near>0.01</near>
-          <far>5</far>
-        </clip>
-      </depth_camera-->
     </camera>
   </sensor>
 </gazebo>
+-->
 </robot>

File: urdf/vx300s_control.xacro (robot description, xacro)
@@ -11,4 +11,5 @@
                     <param name="max">3.14</param-->
                 </command_interface>
+                <command_interface name="velocity"/>
                 <state_interface name="position"/>
                 <state_interface name="velocity"/>
